File: CanLite.kicad_pcb (KiCad board)
At the start: 2 copper layers, 40 x 53.6 mm, 35 parts, among them J1 12V, J2 CAN, J4 Molex_104031-0811, U1 SCT2401, U2 ESP32-WROOM-32D, U3 SN65HVD231

Commit message: Kicad 10 + RevE: protect 5V_prog
Parts:
- added D2: 1N4148, Diode_SMD:D_SOD-323, F.Cu at (112.3, 85.1)
Connections:
- J3 pad 4: /12V_INT -> /5V_prog
Routing:
- net /12V_INT: track 65.4 -> 17.9 mm, vias 1 -> 0
- net /5V_prog: track 0.00 -> 42.4 mm, vias 0 -> 1
Other:
- board text added: "revE"
- board text removed: "revD"
