File: CanLite.kicad_sch (KiCad schematic)
At the start: 36 parts, among them J1 12V, J2 CAN, J2 Molex_104031-0811, U1 SCT2401, U2 ESP32-WROOM-32D, U3 SN65HVD231

Commit message: Kicad 10 + RevE: protect 5V_prog
Parts:
- removed V1: VOLTLOG_LOGO, Voltlog:voltlog_mask_3mm, symbol voltlog:VOLTLOG_LOGO
- added D2: 1N4148, Diode_SMD:D_SOD-323, symbol Diode:1N4148
- J3: value ~ -> (none)
- renumbered J2 to J4, R7 to R10, R12 to R11, R9 to R7, R6 to R8, R5 to R9
Connections:
- net 12V_INT: now also D2.1 (K); no longer J3.4 (Pin_4)
- new net 5V_prog: D2.2 (A), J3.4 (Pin_4)
Other:
- note removed: "VBAT Sense"
